Commit message: Added ccam and ur5 arm specific changes

File: husky_gazebo/urdf/accessories/kinectv2_camera.gazebo.xacro (robot description, xacro)
@@ -1,7 +1,7 @@
 <?xml version="1.0"?>
 <root xmlns:xacro="http://ros.org/wiki/xacro">
-<xacro:macro name="kinect_camera_gazebo" params="prefix">
+<xacro:macro name="kinectv2_camera_gazebo" params="prefix">
   <joint name="${prefix}_optical_joint" type="fixed">
-    <origin xyz="0 0 0" rpy="-1.5708 0 -1.5708"/>
+    <origin xyz="0.0 0.0 0.0" rpy="-1.5708 0 -1.5708"/>
     <parent link="${prefix}_link"/>
     <child link="${prefix}_frame_optical"/>
@@ -11,11 +11,11 @@
     <sensor type="depth" name="${prefix}">
       <always_on>true</always_on>
-      <update_rate>20.0</update_rate>
+      <update_rate>30.0</update_rate>
       <camera>
-        <horizontal_fov>${60.0*M_PI/180.0}</horizontal_fov>
+        <horizontal_fov>${70.0*M_PI/180.0}</horizontal_fov>
         <image>
           <format>R8G8B8</format>
-          <width>640</width>
-          <height>480</height>
+          <width>1920</width>
+          <height>1080</height>
         </image>
         <clip>
@@ -27,5 +27,5 @@
         <cameraName>${prefix}</cameraName>
         <alwaysOn>true</alwaysOn>
-        <updateRate>10</updateRate>
+        <updateRate>30.0</updateRate>
         <imageTopicName>rgb/image_raw</imageTopicName>
         <depthImageTopicName>depth/image_raw</depthImageTopicName>
@@ -35,9 +35,9 @@
         <frameName>${prefix}_frame_optical</frameName>
         <baseline>0.1</baseline>
-        <distortion_k1>0.0</distortion_k1>
-        <distortion_k2>0.0</distortion_k2>
-        <distortion_k3>0.0</distortion_k3>
-        <distortion_t1>0.0</distortion_t1>
-        <distortion_t2>0.0</distortion_t2>
+        <distortionK1>0.0</distortionK1>
+        <distortionK2>0.0</distortionK2>
+        <distortionK3>0.0</distortionK3>
+        <distortionT1>0.0</distortionT1>
+        <distortionT2>0.0</distortionT2>
         <pointCloudCutoff>0.4</pointCloudCutoff>
       </plugin>

File: husky_gazebo/urdf/husky.gazebo.xacro (robot description, xacro)
@@ -23,4 +23,6 @@
 <robot name="husky_robot_gazebo" xmlns:xacro="http://ros.org/wiki/xacro">
   <xacro:include filename="$(find husky_gazebo)/urdf/accessories/kinect_camera.gazebo.xacro"/>
+  <xacro:include filename="$(find husky_gazebo)/urdf/accessories/kinectv2_camera.gazebo.xacro"/>
+  <xacro:include filename="$(find husky_gazebo)/urdf/accessories/basler_camera.gazebo.xacro"/>
   <xacro:macro name="husky_robot_gazebo">
     <gazebo>
@@ -77,7 +79,47 @@
       </gazebo>
     </xacro:if>
+    <xacro:if value="$(arg ur5_camera_enabled)">
+      <!--Remove when https://github.com/ros-industrial/universal_robot/pull/168 is resolved -->
+      <gazebo reference="ur5_arm_shoulder_link">
+        <selfCollide>true</selfCollide>
+      </gazebo>
+      <gazebo reference="ur5_arm_upper_arm_link">
+        <selfCollide>true</selfCollide>
+      </gazebo>
+      <gazebo reference="ur5_arm_forearm_link">
+        <selfCollide>true</selfCollide>
+      </gazebo>
+      <gazebo reference="ur5_arm_wrist_1_link">
+        <selfCollide>true</selfCollide>
+      </gazebo>
+      <gazebo reference="ur5_arm_wrist_3_link">
+       <selfCollide>true</selfCollide>
+      </gazebo>
+      <gazebo reference="ur5_arm_wrist_2_link">
+        <selfCollide>true</selfCollide>
+      </gazebo>
+      <gazebo reference="ur5_arm_ee_link">
+        <selfCollide>true</selfCollide>
+      </gazebo>
+      <gazebo reference="ur5_arm_tool_mount_link">
+        <selfCollide>true</selfCollide>
+      </gazebo>
+      <gazebo reference="ur5_arm_camera_link">
+        <selfCollide>true</selfCollide>
+      </gazebo>
+      <gazebo reference="ur5_arm_marker_link">
+        <selfCollide>true</selfCollide>
+      </gazebo>
+      <xacro:basler_camera_gazebo prefix="ur5_arm_camera"/>
+      <gazebo reference="ur5_arm_camera_frame_optical">
+        <selfCollide>true</selfCollide>
+      </gazebo>
+    </xacro:if>
     <xacro:if value="$(arg kinect_enabled)">
       <xacro:kinect_camera_gazebo prefix="camera"/>
     </xacro:if>
+    <xacro:if value="$(arg kinectv2_enabled)">
+      <xacro:kinectv2_camera_gazebo prefix="camera"/>
+    </xacro:if>
   </xacro:macro>
 </robot>
