Commit message: Removed links from camera gazebo configs and added to individual urdfs

File: husky_gazebo/urdf/accessories/basler_camera.gazebo.xacro (robot description, xacro)
@@ -2,10 +2,4 @@
 <root xmlns:xacro="http://ros.org/wiki/xacro">
 <xacro:macro name="basler_camera_gazebo" params="prefix">
-  <joint name="${prefix}_optical_joint" type="fixed">
-    <origin xyz="0.0 0.0 0.0" rpy="-1.5708 0.0 -1.5708"/>
-    <parent link="${prefix}_link"/>
-    <child link="${prefix}_frame_optical"/>
-  </joint>
-  <link name="${prefix}_frame_optical"/>
   <!-- camera -->
   <gazebo reference="${prefix}_link">
@@ -36,12 +30,13 @@
         <updateRate>150.0</updateRate>
         <cameraName>${prefix}</cameraName>
-        <imageTopicName>image_raw</imageTopicName>
-        <cameraInfoTopicName>camera_info</cameraInfoTopicName>
-        <frameName>${prefix}_frame_optical</frameName>
-        <distortionK1>0.0</distortionK1>
-        <distortionK2>0.0</distortionK2>
-        <distortionK3>0.0</distortionK3>
-        <distortionT1>0.0</distortionT1>
-        <distortionT2>0.0</distortionT2>
+        <imageTopicName>/${prefix}/image_raw</imageTopicName>
+        <cameraInfoTopicName>/${prefix}/camera_info</cameraInfoTopicName>
+        <frameName>${prefix}_optical_frame</frameName>
+	<hackBaseline>0</hackBaseline>
+        <distortion_k1>0.0</distortion_k1>
+        <distortion_k2>0.0</distortion_k2>
+        <distortion_k3>0.0</distortion_k3>
+        <distortion_t1>0.0</distortion_t1>
+        <distortion_t2>0.0</distortion_t2>
       </plugin>
     </sensor>

File: husky_gazebo/urdf/accessories/kinect_camera.gazebo.xacro (robot description, xacro)
@@ -2,10 +2,4 @@
 <root xmlns:xacro="http://ros.org/wiki/xacro">
 <xacro:macro name="kinect_camera_gazebo" params="prefix">
-  <joint name="${prefix}_optical_joint" type="fixed">
-    <origin xyz="0 0 0" rpy="-1.5708 0 -1.5708"/>
-    <parent link="${prefix}_link"/>
-    <child link="${prefix}_frame_optical"/>
-  </joint>
-  <link name="${prefix}_frame_optical"/>
   <gazebo reference="${prefix}_link">
     <sensor type="depth" name="${prefix}">
@@ -27,12 +21,15 @@
         <cameraName>${prefix}</cameraName>
         <alwaysOn>true</alwaysOn>
-        <updateRate>10</updateRate>
-        <imageTopicName>rgb/image_raw</imageTopicName>
-        <depthImageTopicName>depth/image_raw</depthImageTopicName>
-        <pointCloudTopicName>depth/points</pointCloudTopicName>
-        <cameraInfoTopicName>rgb/camera_info</cameraInfoTopicName>
-        <depthImageCameraInfoTopicName>depth/camera_info</depthImageCameraInfoTopicName>
-        <frameName>${prefix}_frame_optical</frameName>
+        <updateRate>20</updateRate>
+        <imageTopicName>/${prefix}/rgb/image_raw</imageTopicName>
+	<cameraInfoTopicName>/${prefix}/rgb/camera_info</cameraInfoTopicName>
+        <depthImageTopicName>/${prefix}/depth/image_raw</depthImageTopicName>
+	<depthImageCameraInfoTopicName>/${prefix}/depth/camera_info</depthImageCameraInfoTopicName>
+        <pointCloudTopicName>/${prefix}/depth/points</pointCloudTopicName>
+        <frameName>${prefix}_optical_frame</frameName>
         <baseline>0.1</baseline>
+        <hackBaseline>0</hackBaseline>
+	<pointCloudCutoff>0.35</pointCloudCutoff>
+        <pointCloudCutoffMax>4.5</pointCloudCutoffMax>
         <distortion_k1>0.0</distortion_k1>
         <distortion_k2>0.0</distortion_k2>
@@ -40,5 +37,4 @@
         <distortion_t1>0.0</distortion_t1>
         <distortion_t2>0.0</distortion_t2>
-        <pointCloudCutoff>0.4</pointCloudCutoff>
       </plugin>
     </sensor>

File: husky_gazebo/urdf/accessories/kinectv2_camera.gazebo.xacro (robot description, xacro)
@@ -2,10 +2,4 @@
 <root xmlns:xacro="http://ros.org/wiki/xacro">
 <xacro:macro name="kinectv2_camera_gazebo" params="prefix">
-  <joint name="${prefix}_optical_joint" type="fixed">
-    <origin xyz="0.0 0.0 0.0" rpy="-1.5708 0 -1.5708"/>
-    <parent link="${prefix}_link"/>
-    <child link="${prefix}_frame_optical"/>
-  </joint>
-  <link name="${prefix}_frame_optical"/>
   <gazebo reference="${prefix}_link">
     <sensor type="depth" name="${prefix}">
@@ -24,21 +18,23 @@
         </clip>
       </camera>
-      <plugin name="kinect_${prefix}_controller" filename="libgazebo_ros_openni_kinect.so">
+      <plugin name="kinectv2_${prefix}_controller" filename="libgazebo_ros_openni_kinect.so">
         <cameraName>${prefix}</cameraName>
         <alwaysOn>true</alwaysOn>
-        <updateRate>30.0</updateRate>
-        <imageTopicName>rgb/image_raw</imageTopicName>
-        <depthImageTopicName>depth/image_raw</depthImageTopicName>
-        <pointCloudTopicName>depth/points</pointCloudTopicName>
-        <cameraInfoTopicName>rgb/camera_info</cameraInfoTopicName>
-        <depthImageCameraInfoTopicName>depth/camera_info</depthImageCameraInfoTopicName>
-        <frameName>${prefix}_frame_optical</frameName>
+        <updateRate>20</updateRate>
+        <imageTopicName>/${prefix}/rgb/image_raw</imageTopicName>
+	<cameraInfoTopicName>/${prefix}/rgb/camera_info</cameraInfoTopicName>
+        <depthImageTopicName>/${prefix}/depth/image_raw</depthImageTopicName>
+	<depthImageCameraInfoTopicName>/${prefix}/depth/camera_info</depthImageCameraInfoTopicName>
+        <pointCloudTopicName>/${prefix}/depth/points</pointCloudTopicName>
+        <frameName>${prefix}_optical_frame</frameName>
         <baseline>0.1</baseline>
-        <distortionK1>0.0</distortionK1>
-        <distortionK2>0.0</distortionK2>
-        <distortionK3>0.0</distortionK3>
-        <distortionT1>0.0</distortionT1>
-        <distortionT2>0.0</distortionT2>
-        <pointCloudCutoff>0.4</pointCloudCutoff>
+	<hackBaseline>0</hackBaseline>
+	<pointCloudCutoff>0.35</pointCloudCutoff>
+        <pointCloudCutoffMax>4.5</pointCloudCutoffMax>
+        <distortion_k1>0.0</distortion_k1>
+        <distortion_k2>0.0</distortion_k2>
+        <distortion_k3>0.0</distortion_k3>
+        <distortion_t1>0.0</distortion_t1>
+        <distortion_t2>0.0</distortion_t2>
       </plugin>
     </sensor>
